File: DC_MOTOR_CONTROLLER/pwm_source.kicad_sch (KiCad schematic)
At the start: 0 parts

Commit message: worked on h-bridge, pwm, io
Parts:
- added C12, C13: C, symbol Device:C
- added D9: MDB8S, Package_SO:TSSOP-4_4.4x5mm_P4mm, symbol Diode_Bridge:MDB8S
- added R4, R5, R6, R7: R, symbol Device:R
- added U4: LM358_DFN, Package_DFN_QFN:DFN-8-1EP_2x2mm_P0.5mm_EP1.05x1.75mm, symbol Amplifier_Operational:LM358_DFN
- added U5: TL331, Package_TO_SOT_SMD:SOT-23-5, symbol Comparator:TL331
- added U6: MCP4725xxx-xCH, Package_TO_SOT_SMD:SOT-23-6, symbol Analog_DAC:MCP4725xxx-xCH
Connections:
- new net: D9.4, R4.1, R7.2, U4.1
- new net: R6.1, R7.1, U4.2 (-)
- new net: C12.2, C13.1, R5.1, U4.3 (+)
- new net: D9.1 (+), U5.3 (+)
- new net: C12.1, R4.2
- new net: U5.1 (-), U6.1 (VOUT)
- new net 5Vdd: U5.5 (V+)
- new net GND: C13.2, D9.2 (-), D9.3, R5.2, R6.2, U5.2 (V-)
