File: DC_MOTOR_CONTROLLER.kicad_sch (KiCad schematic)
At the start: 0 parts

Commit message: Add files via upload
Other:
- sheet io ports: added 3Vdd; removed none
- sheet pwm_source ports: added 5Vdd; removed none
Changed lines of the file:
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@@
+			)
+		)
+		(pin "3Vdd" input
+			(at 111.76 35.56 180)
+			(effects
+				(font
+					(size 1.27 1.27)
+				)
+				(justify left)
 			)
 		)
@@
 			)
 		)
+		(pin "5Vdd" input
+			(at 111.76 90.17 180)
+			(effects
+				(font
+					(size 1.27 1.27)
+				)
+				(justify left)
+			)
+		)
